Commit message: 形を変更

File: nhk2022_simulator/urdf/lidar.urdf.xacro (robot description, xacro)
@@ -1,8 +1,8 @@
 <robot name="lidar" xmlns:xacro="http://ros.org/wiki/xacro">
-  <xacro:macro name="laser_macro" params="parent prefix xyz">
+  <xacro:macro name="laser_macro" params="parent prefix xyz rpy">
     <joint name="${prefix}_joint" type="fixed">
       <parent link="${parent}"/>
       <child  link="${prefix}_link"/>
-      <origin xyz="${xyz}" rpy="0 0 0"/>
+      <origin xyz="${xyz}" rpy="${rpy}"/>
     </joint>
     <link name="${prefix}_link">

File: nhk2022_simulator/urdf/simple_odom_robot.urdf.xacro (robot description, xacro)
@@ -1,5 +1,13 @@
 <?xml version="1.0"?>
 <robot name="odm_robot" xmlns:xacro="http://ros.org/wiki/xacro">
+  <xacro:include filename="$(find nhk2022_simulator)/urdf/lidar.urdf.xacro" />
+  <xacro:include filename="$(find nhk2022_simulator)/urdf/imu.urdf.xacro" />
+  <xacro:property name="PI" value="3.1415926535897931"/>
+  <xacro:property name="b_m" value="5.58"/>
+  <xacro:property name="b_m2" value="${b_m/12}"/><!--for calculation of inertia-->
   <xacro:property name="b_w" value="0.60"/>
+  <xacro:property name="b_h" value="1.20"/>
+  <xacro:property name="b_d" value="0.60"/>
+  <xacro:property name="lidar_w" value="0.64"/>
   <material name="red">
     <color rgba="0.2 0 0 1"/>
@@ -12,22 +20,21 @@
   </joint>
   <link name="body_link">
-   <inertial>
-     <origin xyz="0 0 0.5" rpy="0 0 0"/>
-     <mass value="1"/>
-     <inertia ixx="0.1"  ixy="0"  ixz="0" iyy="0.1" iyz="0" izz="0.1" />
-   </inertial>
-   <visual>
-     <origin xyz="0 0 0" rpy="0 0 0" />
-     <geometry>
-       <cylinder radius="0.1" length="0.1"/>
-     </geometry>
-     <material name="red" />
-   </visual>
-   <collision>
-     <origin xyz="0 0 0" rpy="0 0 0"/>
-     <geometry>
-       <cylinder radius="0.1" length="0.1"/>
-     </geometry>
-   </collision>
+    <visual>
+      <geometry>
+        <box size="${b_d} ${b_w} ${b_h}" />
+      </geometry>
+    </visual>
+    <collision>
+      <geometry>
+          <box size="${b_d*0.95} ${b_w*0.95} ${b_h*0.95}" />
+      </geometry>
+    </collision>
+    <inertial>
+      <origin xyz="0 0 0" rpy="0 0 0" />
+      <mass value="${b_m}" />
+      <inertia ixx="${b_m2*(b_h*b_h+b_w*b_w)}" ixy="0"    ixz="0"
+                iyx="0"   iyy="${b_m2*(b_h*b_h+b_d*b_d)}"  iyz="0"
+                izx="0"   izy="0"  izz="${b_m2*(b_w*b_w+b_d*b_d)}" />
+    </inertial>
   </link>
   <gazebo reference="body_link">
@@ -36,5 +43,5 @@
     <mu2 value="0.1" />
   </gazebo>
-  <joint name="head_joint" type="fixed">
+  <!-- <joint name="head_joint" type="fixed">
     <parent link="base_link"/>
     <child  link="head_link"/>
@@ -42,18 +49,18 @@
   </joint>
   <link name="head_link">
-   <visual>
-     <origin xyz="0 0 0" rpy="0 0 0" />
-     <geometry>
-       <cylinder radius="0.03" length="0.04"/>
-     </geometry>
-     <material name="red" />
-   </visual>
+    <visual>
+      <origin xyz="0 0 0" rpy="0 0 0" />
+      <geometry>
+        <cylinder radius="0.03" length="0.04"/>
+      </geometry>
+      <material name="red" />
+    </visual>
   </link>
   <gazebo reference="head_link">
     <material>Gazebo/Red</material>
-  </gazebo>
-  <xacro:laser_macro prefix="lidar1" parent="base_footprint" xyz="${b_w}/2 ${b_w}/2 0.04" />
-  <xacro:laser_macro prefix="lidar2" parent="base_footprint" xyz="-${b_w}/2 -${b_w}/2 0.04" />
-  <xacro:imu_macro prefix="imu" parent="base_footprint" xyz="0.0 0 0.10" />
+  </gazebo> -->
+  <xacro:laser_macro prefix="lidar1" parent="base_link" xyz="${lidar_w/2} ${lidar_w/2} 0.04" rpy="0 0 ${PI/4}" />
+  <xacro:laser_macro prefix="lidar2" parent="base_link" xyz="-${lidar_w/2} -${lidar_w/2} 0.04" rpy="0 0 -${3*PI/4}" />
+  <xacro:imu_macro prefix="imu" parent="base_link" xyz="0.0 0 0.10" />
   <gazebo>
     <plugin name="object_controller" filename="libgazebo_ros_planar_move.so">

Commit message: 重心を下げないとバグる

File: nhk2022_simulator/urdf/lidar.urdf.xacro (robot description, xacro)
@@ -1,56 +1,57 @@
-<robot name="lidar" xmlns:xacro="http://ros.org/wiki/xacro">
-  <xacro:macro name="laser_macro" params="parent prefix xyz rpy">
-    <joint name="${prefix}_joint" type="fixed">
-      <parent link="${parent}"/>
-      <child  link="${prefix}_link"/>
-      <origin xyz="${xyz}" rpy="${rpy}"/>
-    </joint>
-    <link name="${prefix}_link">
-      <visual>
-        <origin xyz="0 0 0" rpy="0 0 0" />
-        <geometry>
-          <cylinder radius="0.02" length="0.06" />
-        </geometry>
-        <material name="red" />
-      </visual>
-      <collision>
-        <origin xyz="0 0 0" rpy="0 0 0"/>
-        <geometry>
-          <cylinder radius="0.02" length="0.06" />
-        </geometry>
-      </collision>
-    </link>
-    <gazebo reference="${prefix}_link">
-      <material>Gazebo/Red</material>
-      <sensor type="ray" name="${prefix}">
-        <pose>0 0 0 0 0 0</pose>
-        <visualize>false</visualize>
-        <update_rate>10</update_rate>
-        <ray>
-          <scan>
-            <horizontal>
-              <samples>400</samples>
-              <resolution>1</resolution>
-              <min_angle>${radians(-180)}</min_angle>
-              <max_angle>${radians(180)}</max_angle>
-            </horizontal>
-          </scan>
-          <range>
-            <min>0.10</min>
-            <max>20.0</max>
-            <resolution>0.01</resolution>
-          </range>
-          <noise>
-            <type>gaussian</type>
-            <mean>0.0</mean>
-            <stddev>0.01</stddev>
-          </noise>
-        </ray>
-        <plugin name="gazebo_ros_lidar_controller" filename="libgazebo_ros_laser.so">
-          <topicName>/scan</topicName>
-          <frameName>${prefix}_link</frameName>
-        </plugin>
-      </sensor>
-    </gazebo>
-  </xacro:macro>
+<robot name="lidar"
+    xmlns:xacro="http://ros.org/wiki/xacro">
+    <xacro:macro name="laser_macro" params="parent prefix xyz rpy">
+        <joint name="${prefix}_joint" type="fixed">
+            <parent link="${parent}"/>
+            <child link="${prefix}_link"/>
+            <origin xyz="${xyz}" rpy="${rpy}"/>
+        </joint>
+        <link name="${prefix}_link">
+            <visual>
+                <origin xyz="0 0 0" rpy="0 0 0" />
+                <geometry>
+                    <cylinder radius="0.02" length="0.06" />
+                </geometry>
+                <material name="red" />
+            </visual>
+            <collision>
+                <origin xyz="0 0 0" rpy="0 0 0"/>
+                <geometry>
+                    <cylinder radius="0.02" length="0.06" />
+                </geometry>
+            </collision>
+        </link>
+        <gazebo reference="${prefix}_link">
+            <material>Gazebo/Red</material>
+            <sensor type="ray" name="${prefix}">
+                <pose>0 0 0 0 0 0</pose>
+                <visualize>false</visualize>
+                <update_rate>10</update_rate>
+                <ray>
+                    <scan>
+                        <horizontal>
+                            <samples>400</samples>
+                            <resolution>1</resolution>
+                            <min_angle>${radians(-180)}</min_angle>
+                            <max_angle>${radians(180)}</max_angle>
+                        </horizontal>
+                    </scan>
+                    <range>
+                        <min>0.10</min>
+                        <max>20.0</max>
+                        <resolution>0.01</resolution>
+                    </range>
+                    <noise>
+                        <type>gaussian</type>
+                        <mean>0.0</mean>
+                        <stddev>0.01</stddev>
+                    </noise>
+                </ray>
+                <plugin name="gazebo_ros_lidar_controller" filename="libgazebo_ros_laser.so">
+                    <topicName>/scan</topicName>
+                    <frameName>${prefix}_link</frameName>
+                </plugin>
+            </sensor>
+        </gazebo>
+    </xacro:macro>
 </robot>

File: nhk2022_simulator/urdf/simple_odom_robot.urdf.xacro (robot description, xacro)
@@ -1,49 +1,49 @@
 <?xml version="1.0"?>
-<robot name="odm_robot" xmlns:xacro="http://ros.org/wiki/xacro">
-  <xacro:include filename="$(find nhk2022_simulator)/urdf/lidar.urdf.xacro" />
-  <xacro:include filename="$(find nhk2022_simulator)/urdf/imu.urdf.xacro" />
-  <xacro:property name="PI" value="3.1415926535897931"/>
-  <xacro:property name="b_m" value="5.58"/>
-  <xacro:property name="b_m2" value="${b_m/12}"/><!--for calculation of inertia-->
-  <xacro:property name="b_w" value="0.60"/>
-  <xacro:property name="b_h" value="1.20"/>
-  <xacro:property name="b_d" value="0.60"/>
-  <xacro:property name="lidar_w" value="0.64"/>
-  <material name="red">
-    <color rgba="0.2 0 0 1"/>
-  </material>
-  <link name="base_link"/>
-  <joint name="body_joint" type="fixed">
+<robot name="odm_robot"
+    xmlns:xacro="http://ros.org/wiki/xacro">
+    <xacro:include filename="$(find nhk2022_simulator)/urdf/lidar.urdf.xacro" />
+    <xacro:include filename="$(find nhk2022_simulator)/urdf/imu.urdf.xacro" />
+    <xacro:property name="PI" value="3.1415926535897931"/>
+    <xacro:property name="b_m" value="5.58"/>
+    <xacro:property name="b_m2" value="${b_m/12}"/>
+    <!--for calculation of inertia-->
+    <xacro:property name="b_w" value="0.60"/>
+    <xacro:property name="b_h" value="0.1"/>
+    <xacro:property name="b_d" value="0.60"/>
+    <xacro:property name="lidar_w" value="0.64"/>
+    <material name="red">
+        <color rgba="0.2 0 0 1"/>
+    </material>
+    <link name="base_link"/>
+    <joint name="body_joint" type="fixed">
+        <parent link="base_link"/>
+        <child link="body_link"/>
+        <origin xyz="0 0 ${b_h/2}" rpy="0 0 0"/>
+    </joint>
+    <link name="body_link">
+        <visual>
+            <geometry>
+                <box size="${b_d} ${b_w} ${b_h}" />
+            </geometry>
+        </visual>
+        <collision>
+            <geometry>
+                <box size="${b_d*0.95} ${b_w*0.95} ${b_h*0.95}" />
+            </geometry>
+        </collision>
+        <inertial>
+            <origin xyz="0 0 0" rpy="0 0 0" />
+            <mass value="${b_m}" />
+            <inertia ixx="${b_m2*(b_h*b_h+b_w*b_w)}" ixy="0" ixz="0" iyx="0" iyy="${b_m2*(b_h*b_h+b_d*b_d)}" iyz="0" izx="0" izy="0" izz="${b_m2*(b_w*b_w+b_d*b_d)}" />
+        </inertial>
+    </link>
+    <gazebo reference="body_link">
+        <material>Gazebo/Red</material>
+        <mu1 value="0.1" />
+        <mu2 value="0.1" />
+    </gazebo>
+    <!-- <joint name="head_joint" type="fixed">
     <parent link="base_link"/>
-    <child  link="body_link"/>
-    <origin xyz="0 0 ${b_h/2}" rpy="0 0 0"/>
-  </joint>
-  <link name="body_link">
-    <visual>
-      <geometry>
-        <box size="${b_d} ${b_w} ${b_h}" />
-      </geometry>
-    </visual>
-    <collision>
-      <geometry>
-          <box size="${b_d*0.95} ${b_w*0.95} ${b_h*0.95}" />
-      </geometry>
-    </collision>
-    <inertial>
-      <origin xyz="0 0 0" rpy="0 0 0" />
-      <mass value="${b_m}" />
-      <inertia ixx="${b_m2*(b_h*b_h+b_w*b_w)}" ixy="0"    ixz="0"
-                iyx="0"   iyy="${b_m2*(b_h*b_h+b_d*b_d)}"  iyz="0"
-                izx="0"   izy="0"  izz="${b_m2*(b_w*b_w+b_d*b_d)}" />
-    </inertial>
-  </link>
-  <gazebo reference="body_link">
-    <material>Gazebo/Red</material>
-    <mu1 value="0.1" />
-    <mu2 value="0.1" />
-  </gazebo>
-  <!-- <joint name="head_joint" type="fixed">
-    <parent link="base_link"/>
-    <child  link="head_link"/>
+    <child link="head_link"/>
     <origin xyz="0.05 0 0.12" rpy="0 0 0"/>
   </joint>
@@ -60,16 +60,16 @@
     <material>Gazebo/Red</material>
   </gazebo> -->
-  <xacro:laser_macro prefix="lidar1" parent="base_link" xyz="${lidar_w/2} ${lidar_w/2} 0.04" rpy="0 0 ${PI/4}" />
-  <xacro:laser_macro prefix="lidar2" parent="base_link" xyz="-${lidar_w/2} -${lidar_w/2} 0.04" rpy="0 0 -${3*PI/4}" />
-  <xacro:imu_macro prefix="imu" parent="base_link" xyz="0.0 0 0.10" />
-  <gazebo>
-    <plugin name="object_controller" filename="libgazebo_ros_planar_move.so">
-      <commandTopic>cmd_vel</commandTopic>
-      <odometryTopic>odom</odometryTopic>
-      <odometryFrame>odom</odometryFrame>
-      <odometryRate>20.0</odometryRate>
-      <robotBaseFrame>base_link</robotBaseFrame>
-      <cmdTimeout>2.0</cmdTimeout>
-    </plugin>
-  </gazebo>
+    <xacro:laser_macro prefix="lidar1" parent="base_link" xyz="${lidar_w/2} ${lidar_w/2} 0.04" rpy="0 0 ${PI/4}" />
+    <xacro:laser_macro prefix="lidar2" parent="base_link" xyz="-${lidar_w/2} -${lidar_w/2} 0.04" rpy="0 0 -${3*PI/4}" />
+    <xacro:imu_macro prefix="imu" parent="base_link" xyz="0.0 0 0.10" />
+    <gazebo>
+        <plugin name="object_controller" filename="libgazebo_ros_planar_move.so">
+            <commandTopic>cmd_vel</commandTopic>
+            <odometryTopic>odom</odometryTopic>
+            <odometryFrame>odom</odometryFrame>
+            <odometryRate>20.0</odometryRate>
+            <robotBaseFrame>base_link</robotBaseFrame>
+            <cmdTimeout>2.0</cmdTimeout>
+        </plugin>
+    </gazebo>
 </robot>
