Commit message: 一旦スポーン完了

File: nhk2022_simulator/urdf/simple_odom_robot.urdf.xacro (robot description, xacro)
@@ -1,4 +1,5 @@
 <?xml version="1.0"?>
 <robot name="odm_robot" xmlns:xacro="http://ros.org/wiki/xacro">
+  <xacro:property name="b_w" value="0.60"/>
   <material name="red">
     <color rgba="0.2 0 0 1"/>
@@ -52,4 +53,7 @@
     <material>Gazebo/Red</material>
   </gazebo>
+  <xacro:laser_macro prefix="lidar1" parent="base_footprint" xyz="${b_w}/2 ${b_w}/2 0.04" />
+  <xacro:laser_macro prefix="lidar2" parent="base_footprint" xyz="-${b_w}/2 -${b_w}/2 0.04" />
+  <xacro:imu_macro prefix="imu" parent="base_footprint" xyz="0.0 0 0.10" />
   <gazebo>
     <plugin name="object_controller" filename="libgazebo_ros_planar_move.so">

Commit message: 高さ方向を修正

File: nhk2022_simulator/urdf/simple_odom_robot.urdf.xacro (robot description, xacro)
@@ -17,5 +17,5 @@
     <parent link="base_link"/>
     <child  link="body_link"/>
-    <origin xyz="0 0 0.05" rpy="0 0 0"/>
+    <origin xyz="0 0 ${b_h/2}" rpy="0 0 0"/>
   </joint>
   <link name="body_link">

Commit message: 質量も追加で。

File: nhk2022_simulator/urdf/simple_odom_robot.urdf.xacro (robot description, xacro)
@@ -5,5 +5,5 @@
     <xacro:include filename="$(find nhk2022_simulator)/urdf/imu.urdf.xacro" />
     <xacro:property name="PI" value="3.1415926535897931"/>
-    <xacro:property name="b_m" value="5.58"/>
+    <xacro:property name="b_m" value="20.0"/>
     <xacro:property name="b_m2" value="${b_m/12}"/>
     <!--for calculation of inertia-->
