Commit message: lidar角度調整

File: nhk2022_launcher/urdf/R2.urdf (robot description, URDF)
Before this commit: robot R2, 3 links, 2 joints
Joints:
- joint laser_link_joint: origin xyz=-0.16 0.0 0.0 rpy=0 -0 0 -> xyz=0.16 0.16 0.0 rpy=0 -0 0

Commit message: slamのlaunchを編集

File: nhk2022_launcher/urdf/R2.urdf (robot description, URDF)
Before this commit: robot R2, 3 links, 2 joints
Links:
- removed link laser
- added link laser1
- added link laser2
Joints:
- removed joint laser_link_joint
- added joint laser1_link_joint: type fixed, parent base_footprint, child laser1, origin xyz=0.16 0.16 0.0 rpy=0 -0 0
- added joint laser2_link_joint: type fixed, parent base_footprint, child laser2, origin xyz=0.16 0.16 0.0 rpy=0 -0 0

Commit message: gmapping あまりうまく行かず。

File: nhk2022_launcher/urdf/R2.urdf (robot description, URDF)
Before this commit: robot R2, 4 links, 3 joints
Joints:
- joint imu_link_joint: origin xyz=0.0 0.0 0.0 rpy=0 -0 0 -> xyz=0.0 0.0 0.0 rpy=0 -0 3.1415
- joint laser1_link_joint: origin xyz=0.16 0.16 0.0 rpy=0 -0 0 -> xyz=0.48 0.48 0.0 rpy=0 -0 0.785
- joint laser2_link_joint: origin xyz=0.16 0.16 0.0 rpy=0 -0 0 -> xyz=-0.48 -0.48 0.0 rpy=0 -0 -2.355

Commit message: teleopの復活

File: nhk2022_launcher/urdf/R2.urdf (robot description, URDF)
Before this commit: robot R2, 4 links, 3 joints
Joints:
- joint imu_link_joint: origin xyz=0.0 0.0 0.0 rpy=0 -0 3.1415 -> xyz=0.0 0.0 0.3 rpy=0 -0 3.1415
- joint laser1_link_joint: origin xyz=0.48 0.48 0.0 rpy=0 -0 0.785 -> xyz=0.48 -0.48 0.0 rpy=0 -0 -0.785
- joint laser2_link_joint: origin xyz=-0.48 -0.48 0.0 rpy=0 -0 -2.355 -> xyz=-0.48 0.48 0.0 rpy=0 -0 2.355

Commit message: パラメータ調整完了

File: nhk2022_launcher/urdf/R2.urdf (robot description, URDF)
Before this commit: robot R2, 4 links, 3 joints
Joints:
- joint imu_link_joint: origin xyz=0.0 0.0 0.3 rpy=0 -0 3.1415 -> xyz=0.0 0.0 0.3 rpy=0 00 0

Commit message: 車幅パラメータ調整済み

File: nhk2022_launcher/urdf/R2.urdf (robot description, URDF)
Before this commit: robot R2, 4 links, 3 joints
Joints:
- joint laser1_link_joint: origin xyz=0.48 -0.48 0.0 rpy=0 -0 -0.785 -> xyz=0.315 -0.315 0.0 rpy=0 -0 -0.785
- joint laser2_link_joint: origin xyz=-0.48 0.48 0.0 rpy=0 -0 2.355 -> xyz=-0.315 0.315 0.0 rpy=0 -0 2.355
