Commit message: changed some names to R1

File: nhk2022_launcher/urdf/R1.urdf (robot description, URDF)
Before this commit: robot DR, 3 links, 2 joints
Joints:
- joint laser_link_joint: origin xyz=-0.16 0.0 0.0 rpy=0 -0 0 -> xyz=0.37 0.0 0.0 rpy=0 -0 0

File: nhk2022_launcher/urdf/R2.urdf (robot description, URDF)
Before this commit: robot TR, 3 links, 2 joints
Joints:
- joint laser_link_joint: origin xyz=0.37 0.0 0.0 rpy=0 -0 0 -> xyz=-0.16 0.0 0.0 rpy=0 -0 0

Commit message: base_footprintをbase_linkに変更

File: nhk2022_launcher/urdf/R1.urdf (robot description, URDF)
Before this commit: robot R1, 3 links, 2 joints
Links:
- removed link base_footprint
- added link base_link
Joints:
- joint imu_link_joint: parent base_footprint -> base_link
- joint laser_link_joint: parent base_footprint -> base_link

File: nhk2022_launcher/urdf/R2.urdf (robot description, URDF)
Before this commit: robot R2, 4 links, 3 joints
Links:
- removed link base_footprint
- added link base_link
Joints:
- joint imu_link_joint: parent base_footprint -> base_link
- joint laser1_link_joint: parent base_footprint -> base_link
- joint laser2_link_joint: parent base_footprint -> base_link

File: nhk2022_simulator/urdf/omni_body.urdf.xacro (robot description, xacro)
@@ -1,8 +1,8 @@
 <?xml version="1.0" ?>
 <robot name="body" xmlns:xacro="http://ros.org/wiki/xacro">
-   <link name="base_footprint" />
+   <link name="base_link" />
    <link name="base_link" />
    <joint name="base_joint" type="fixed">
-   <parent link="base_footprint" />
+   <parent link="base_link" />
       <child link="base_link" />
       <origin xyz="0 0 0.01" rpy="0 0 0" />
@@ -33,5 +33,5 @@
    </link>
    <joint name="body_joint" type="fixed">
-   <parent link="base_footprint" />
+   <parent link="base_link" />
       <child link="body" />
       <origin xyz="0 0 0.195" rpy="0 0 0" />

File: nhk2022_simulator/urdf/omni_robot.urdf.xacro (robot description, xacro)
@@ -5,9 +5,9 @@
     <xacro:include filename="$(find nhk2022_simulator)/urdf/lidar.urdf.xacro" />
     <xacro:include filename="$(find nhk2022_simulator)/urdf/imu.urdf.xacro" />
-    <xacro:laser_macro prefix="rplidar" parent="base_footprint" xyz="0.23 0 0.04" />
-    <xacro:imu_macro prefix="imu" parent="base_footprint" xyz="0.0 0 0.10" />
-    <xacro:wheel rl="rf" parent="base_footprint" />
-    <xacro:wheel rl="lf" parent="base_footprint" />
-    <xacro:wheel rl="rb" parent="base_footprint" />
-    <xacro:wheel rl="lb" parent="base_footprint" />
+    <xacro:laser_macro prefix="rplidar" parent="base_link" xyz="0.23 0 0.04" />
+    <xacro:imu_macro prefix="imu" parent="base_link" xyz="0.0 0 0.10" />
+    <xacro:wheel rl="rf" parent="base_link" />
+    <xacro:wheel rl="lf" parent="base_link" />
+    <xacro:wheel rl="rb" parent="base_link" />
+    <xacro:wheel rl="lb" parent="base_link" />
 </robot>

Commit message: iroiroparame-ta

File: nhk2022_launcher/urdf/R1.urdf (robot description, URDF)
Before this commit: robot R1, 3 links, 2 joints
Joints:
- joint laser_link_joint: origin xyz=0.37 0.0 0.0 rpy=0 -0 0 -> xyz=0.0 0.0 0.0 rpy=0 -0 0
